File: reviung/41_1350 choc hotswappable/41_1350_pcb/41_1350_pcb.kicad_pcb (KiCad board)
At the start: 2 copper layers, 238.7 x 95.3 mm, 91 parts, among them J3 Pimoroni, U1 ProMicro

Commit message: reviung41: add choc hotswappable (v0.2)
Parts:
- removed Kailh PG1350: Choc, keeblib:Kailh-PG1350-2uStabilizer
- added ?: , , F.Cu at (211.8, 92.5)
- added ?: , , F.Cu at (177.4, 103.7)
- added ?: , , F.Cu at (170.0, 71.6)
- added ?: , , F.Cu at (204.1, 59.1)
- added ?: , , B.Cu at (121.4, 103.7)
- added ?: , , B.Cu at (94.6, 59.1)
- added ?: , , B.Cu at (87.0, 92.5)
- added ?: , , B.Cu at (128.7, 71.6)
- added REF**: grid, 41_1350:grid, B.Cu at (59.1, 61.7)
- added REF**: grid, 41_1350:grid, B.Cu at (63.3, 85.1)
- added REF**: M2_HOLE_NPH, holykeebs:M2_HOLE_NPH, B.Cu at (57.7, 59.0)
- added REF**: M2_HOLE_NPH, holykeebs:M2_HOLE_NPH, F.Cu at (248.5, 91.8)
- added REF**: M2_HOLE_NPH, holykeebs:M2_HOLE_NPH, F.Cu at (241.0, 59.0)
- added REF**: M2_HOLE_NPH, holykeebs:M2_HOLE_NPH, F.Cu at (165.6, 129.5)
- added REF**: M2_HOLE_NPH, holykeebs:M2_HOLE_NPH, B.Cu at (133.1, 129.5)
- added REF**: M2_HOLE_NPH, holykeebs:M2_HOLE_NPH, B.Cu at (50.2, 91.8)
- REF** (x2): moved to F.Cu
- moved REF** 100.6 mm to (195.6, 72.1)
- moved REF** 92.1 mm to (191.3, 95.5), turned to 0 degrees
- moved RSW1 5.44 mm to (170.6, 48.5)
Routing:
- net col1: track 325.5 -> 393.8 mm
- net rowG: track 132.6 -> 198.6 mm
- net col2: track 313.3 -> 368.9 mm
- net col0: track 394.9 -> 399.8 mm
- net GND: track 92.9 -> 88.2 mm
- net Net-(D_E3-A): track 12.2 -> 16.1 mm
- net RST: track 37.4 -> 33.9 mm
- net rowF: track 180.9 -> 183.2 mm
- net rowB: track 133.6 -> 135.8 mm
- net col4: track 351.7 -> 353.7 mm
- net col5: track 306.6 -> 307.9 mm
- net rowA: track 130.7 -> 131.5 mm
- net rowC: track 147.1 -> 147.7 mm
Other:
- board text added: "github.com/idank/keyboards v0.2"
- board text removed: "original design by gtips github.com/idank/keyboards v0.1"
