File: reviung/lowprofile_41_1353/pcb/r41l2.kicad_pcb (KiCad board)
At the start: 2 copper layers, 251.3 x 103.7 mm, 89 parts, among them J3 Pimoroni, SW01 SW_SPDT, U1 ProMicro

Commit message: reviung41: add choc hotswappable (v0.2)
Parts:
- added J2: PIM, pimoroni:pim447, F.Cu at (150.8, 34.6)
- D_A0, D_A1, D_A2, D_A3, D_A4, D_A5, D_B0, D_B1, D_B2, D_B3, D_B4, D_B5, D_C0, D_C1, D_C2, D_C3, D_C4, D_C5, D_D0, D_D1, D_D2, D_D3, D_D4, D_D5, D_E0, D_E1, D_E2, D_E3, D_E4, D_E5, D_F0, D_F1, D_F2, D_F3, D_F4, D_F5, D_G0, D_G1, D_G2, D_G3, D_G4: footprint keeblib:D_MiniMELF_bsides -> kbd:D3_SMD_v2
- SwA0, SwA1, SwA2, SwA3, SwA4, SwA5, SwB0, SwB1, SwB2, SwB3, SwB4, SwB5, SwC0, SwC1, SwC2, SwC3, SwC4, SwC5, SwD0, SwD1, SwD2, SwD3, SwD4, SwD5, SwE0, SwE1, SwE2, SwE3, SwE4, SwE5, SwF0, SwF1, SwF2, SwF3, SwF4, SwF5, SwG0, SwG1, SwG3, SwG4: footprint keeblib:pg1353 -> keyswitches:SW_PG1350
- SwG2: footprint keeblib:pg1353_2u -> keyswitches:SW_PG1350
Routing:
- net col3: track 277.9 -> 349.4 mm
- net col0: track 332.0 -> 402.9 mm
- net col1: track 304.7 -> 375.2 mm
- net col4: track 281.6 -> 350.9 mm
- net col5: track 221.5 -> 282.9 mm
- net col2: track 295.2 -> 356.6 mm
- net Net-(D_D0-Pad2): track 10.7 -> 0.00 mm
- net Net-(D_G3-Pad2): track 10.7 -> 0.00 mm
- net Net-(D_F0-Pad2): track 10.7 -> 0.00 mm
- net Net-(D_F2-Pad2): track 10.5 -> 0.00 mm
- net Net-(D_D2-Pad2): track 10.5 -> 0.00 mm
- net Net-(D_E2-Pad2): track 10.5 -> 0.00 mm
- net Net-(D_G1-Pad2): track 10.4 -> 0.00 mm
- net Net-(D_F5-Pad2): track 10.3 -> 0.00 mm
- net Net-(D_D5-Pad2): track 10.3 -> 0.00 mm
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