File: reviung/reviung41 choc/pcb/reviung41 choc.kicad_pcb (KiCad board)
At the start: 2 copper layers, 238.7 x 95.3 mm, 101 parts, among them SW1 SW_PUSH, SW10 SW_PUSH, SW11 SW_PUSH, SW12 SW_PUSH, SW13 SW_PUSH, SW14 SW_PUSH, SW15 SW_PUSH, SW16 SW_PUSH, SW17 SW_PUSH, SW18 SW_PUSH, SW19 SW_PUSH, SW2 SW_PUSH, SW20 SW_PUSH, SW21 SW_PUSH, SW22 SW_PUSH, SW23 SW_PUSH, SW24 SW_PUSH, SW25 SW_PUSH, SW26 SW_PUSH, SW27 SW_PUSH, SW28 SW_PUSH, SW29 SW_PUSH, SW3 SW_PUSH, SW30 SW_PUSH, SW31 SW_PUSH, SW32 SW_PUSH, SW33 SW_PUSH, SW34 SW_PUSH, SW35 SW_PUSH, SW36 SW_PUSH, SW37 SW_PUSH, SW38 SW_PUSH, SW39 SW_2U_PUSH, SW4 SW_PUSH, SW40 SW_PUSH, SW41 SW_PUSH, SW5 SW_PUSH, SW6 SW_PUSH, SW7 SW_PUSH, SW8 SW_PUSH, SW9 SW_PUSH, U1 ProMicro

Commit message: reviung41: update version
Other:
- board text added: "reviung41 choc github.com/idank/keyboards@fd87392"
- board text removed: "reviung41 choc, v0.3 github.com/idank/keyboards"
Changed lines of the file:
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@@
     (fp_arc (start 37.146773 3.355529) (mid 36.696871 3.406789) (end 36.246969 3.355529)
       (stroke (width 0.2) (type solid)) (layer "Edge.Cuts"))
-    (fp_arc (start 39.503394 81.579917) (mid 39.236234 82.062185) (end 38.753975 82.329336)
+    (fp_arc (start 39.503394 81.579917) (mid 39.236249 82.0622) (end 38.753975 82.329336)
       (stroke (width 0.2) (type solid)) (layer "Edge.Cuts"))
     (fp_arc (start 40.441672 77.515789) (mid 40.793521 76.958127) (end 41.416042 76.74074)
       (stroke (width 0.2) (type solid)) (layer "Edge.Cuts"))
-    (fp_arc (start 49.460861 0.512599) (mid 51.695818 0.128567) (end 53.959882 0)
+    (fp_arc (start 49.460861 0.512599) (mid 51.695818 0.128562) (end 53.959882 0)
       (stroke (width 0.2) (type solid)) (layer "Edge.Cuts"))
     (fp_arc (start 56.605052 60.530052) (mid 56.822458 59.907551) (end 57.380101 59.555682)
@@
     (fp_arc (start 103.255743 53.229393) (mid 101.020785 53.613422) (end 98.756722 53.741992)
       (stroke (width 0.2) (type solid)) (layer "Edge.Cuts"))
-    (fp_arc (start 107.332459 0) (mid 107.954995 0.217376) (end 108.30683 0.775048)
+    (fp_arc (start 107.332459 0) (mid 107.954971 0.217385) (end 108.30683 0.775048)
       (stroke (width 0.2) (type solid)) (layer "Edge.Cuts"))
-    (fp_arc (start 119.323515 48.493552) (mid 119.197193 49.248429) (end 118.574096 49.692873)
+    (fp_arc (start 119.323515 48.493552) (mid 119.19719 49.24841) (end 118.574096 49.692873)
       (stroke (width 0.2) (type solid)) (layer "Edge.Cuts"))
   )
@@
     (pad "" np_thru_hole circle (at 0 0 180) (size 2.3 2.3) (drill 2.3) (layers "*.Cu" "*.Mask"))
   )
-  (gr_text "reviung41 choc, v0.3\ngithub.com/idank/keyboards" (at 161.862222 52.8 -13) (layer "B.SilkS")
-    (effects (font (size 1 1.3) (thickness 0.2)) (justify left mirror))
+  (gr_text "reviung41 choc\ngithub.com/idank/keyboards@fd87392" (at 149.952222 49.75 347) (layer "B.SilkS")
+    (effects (font (size 1 1.2) (thickness 0.2)) (justify mirror))
   )
   (segment (start 156.957411 70.534811) (end 157.072222 70.42) (width 0.25) (layer "F.Cu") (net 1))
