File: corne/corne-light-smt/corne-light.kicad_sch (KiCad schematic)
At the start: 92 parts, among them J1 MJ-4PP-9, J2 OLED, J6 MJ-4PP-9, J7 OLED, SW1 SW_PUSH, SW10 SW_PUSH, SW11 SW_PUSH, SW12 SW_PUSH, SW13 SW_PUSH, SW14 SW_PUSH, SW15 SW_PUSH, SW16 SW_PUSH, SW17 SW_PUSH, SW18 SW_PUSH, SW19 SW_PUSH, SW2 SW_PUSH, SW20 SW_PUSH, SW21 SW_PUSH, SW22 SW_PUSH, SW23 SW_PUSH, SW24 SW_PUSH, SW25 SW_PUSH, SW26 SW_PUSH, SW27 SW_PUSH, SW28 SW_PUSH, SW29 SW_PUSH, SW3 SW_PUSH, SW30 SW_PUSH, SW31 SW_PUSH, SW32 SW_PUSH, SW33 SW_PUSH, SW34 SW_PUSH, SW35 SW_PUSH, SW36 SW_PUSH, SW37 SW_PUSH, SW38 SW_PUSH, SW39 SW_PUSH, SW4 SW_PUSH, SW40 SW_PUSH, SW41 SW_PUSH, SW42 SW_PUSH, SW5 SW_PUSH, SW6 SW_PUSH, SW7 SW_PUSH, SW8 SW_PUSH, SW9 SW_PUSH, U1 ProMicro, U2 ProMicro

Commit message: corne-light-smt: initial version
Parts:
- added BACKLED1, BACKLED10, BACKLED11, BACKLED12, BACKLED13, BACKLED14, BACKLED15, BACKLED16, BACKLED17, BACKLED18, BACKLED2, BACKLED3, BACKLED4, BACKLED5, BACKLED6, BACKLED7, BACKLED8, BACKLED9, BACKLEDr1, BACKLEDr10, BACKLEDr11, BACKLEDr12, BACKLEDr13, BACKLEDr14, BACKLEDr15, BACKLEDr16, BACKLEDr17, BACKLEDr18, BACKLEDr2, BACKLEDr3, BACKLEDr4, BACKLEDr5, BACKLEDr6, BACKLEDr7, BACKLEDr8, BACKLEDr9: SK6805-EC15, holykeebs:LED_SK6805-EC15_1.5x1.5mm_P0.6mm_handsolder, symbol sk6805-ec15:SK6805-EC15
- added C1, C2: 1µ, Capacitor_SMD:C_0402_1005Metric, symbol Device:C
- added L1, L10, L11, L12, L13, L14, L15, L16, L17, L18, L19, L2, L20, L21, L28, L29, L3, L30, L31, L32, L33, L34, L35, L36, L37, L38, L39, L4, L40, L41, L42, L43, L44, L45, L46, L47, L48, L5, L6, L7, L8, L9: SK6812MINI, PCM_marbastlib-various:LED_6028R, symbol PCM_marbastlib-various:SK6812MINI-E
- D1, D10, D11, D12, D13, D14, D15, D16, D17, D18, D19, D2, D20, D21, D22, D23, D24, D25, D26, D27, D28, D29, D3, D30, D31, D32, D33, D34, D35, D36, D37, D38, D39, D4, D40, D41, D42, D5, D6, D7, D8, D9: footprint kbd:D3_TH -> kbd:D3_SMD_v2
- SW1, SW10, SW11, SW12, SW13, SW14, SW15, SW16, SW17, SW18, SW19, SW2, SW20, SW3, SW4, SW5, SW6, SW7, SW8, SW9: footprint kbd:CherryMX_ChocV2_1u -> holykeebs:SW_choc_v1_HS_CPG135001S30_1u
- SW21, SW42: footprint kbd:CherryMX_ChocV2_1.5u -> PCM_marbastlib-choc:SW_choc_v1_HS_CPG135001S30_1.5u
- SW22, SW23, SW24, SW25, SW26, SW27, SW28, SW29, SW30, SW31, SW32, SW33, SW34, SW35, SW36, SW37, SW38, SW39, SW40, SW41: footprint kbd:CherryMX_ChocV2_1u -> holykeebs:SW_choc_v1_HS_CPG135001S30_1u_flipped
- U1, U2: footprint kbd:ProMicro_v3 -> holykeebs:ProMicro_1mm_holes
Connections:
- net GND: now also BACKLED1.4 (GND), BACKLED10.4 (GND), BACKLED11.4 (GND), BACKLED12.4 (GND), BACKLED13.4 (GND), BACKLED14.4 (GND), BACKLED15.4 (GND), BACKLED16.4 (GND), BACKLED17.4 (GND), BACKLED18.4 (GND), BACKLED2.4 (GND), BACKLED3.4 (GND), BACKLED4.4 (GND), BACKLED5.4 (GND), BACKLED6.4 (GND), BACKLED7.4 (GND), BACKLED8.4 (GND), BACKLED9.4 (GND), C1.2, L1.4 (VSS), L10.4 (VSS), L11.4 (VSS), L12.4 (VSS), L13.4 (VSS), L14.4 (VSS), L15.4 (VSS), L16.4 (VSS), L17.4 (VSS), L18.4 (VSS), L19.4 (VSS), L2.4 (VSS), L20.4 (VSS), L21.4 (VSS), L3.4 (VSS), L4.4 (VSS), L5.4 (VSS), L6.4 (VSS), L7.4 (VSS), L8.4 (VSS), L9.4 (VSS)
- net GNDA: now also BACKLEDr1.4 (GND), BACKLEDr10.4 (GND), BACKLEDr11.4 (GND), BACKLEDr12.4 (GND), BACKLEDr13.4 (GND), BACKLEDr14.4 (GND), BACKLEDr15.4 (GND), BACKLEDr16.4 (GND), BACKLEDr17.4 (GND), BACKLEDr18.4 (GND), BACKLEDr2.4 (GND), BACKLEDr3.4 (GND), BACKLEDr4.4 (GND), BACKLEDr5.4 (GND), BACKLEDr6.4 (GND), BACKLEDr7.4 (GND), BACKLEDr8.4 (GND), BACKLEDr9.4 (GND), C2.2, L28.4 (VSS), L29.4 (VSS), L30.4 (VSS), L31.4 (VSS), L32.4 (VSS), L33.4 (VSS), L34.4 (VSS), L35.4 (VSS), L36.4 (VSS), L37.4 (VSS), L38.4 (VSS), L39.4 (VSS), L40.4 (VSS), L41.4 (VSS), L42.4 (VSS), L43.4 (VSS), L44.4 (VSS), L45.4 (VSS), L46.4 (VSS), L47.4 (VSS), L48.4 (VSS)
- net VCC: now also BACKLED1.2 (VDD), BACKLED10.2 (VDD), BACKLED11.2 (VDD), BACKLED12.2 (VDD), BACKLED13.2 (VDD), BACKLED14.2 (VDD), BACKLED15.2 (VDD), BACKLED16.2 (VDD), BACKLED17.2 (VDD), BACKLED18.2 (VDD), BACKLED2.2 (VDD), BACKLED3.2 (VDD), BACKLED4.2 (VDD), BACKLED5.2 (VDD), BACKLED6.2 (VDD), BACKLED7.2 (VDD), BACKLED8.2 (VDD), BACKLED9.2 (VDD), C1.1, L1.1 (VDD), L10.1 (VDD), L11.1 (VDD), L12.1 (VDD), L13.1 (VDD), L14.1 (VDD), L15.1 (VDD), L16.1 (VDD), L17.1 (VDD), L18.1 (VDD), L19.1 (VDD), L2.1 (VDD), L20.1 (VDD), L21.1 (VDD), L3.1 (VDD), L4.1 (VDD), L5.1 (VDD), L6.1 (VDD), L7.1 (VDD), L8.1 (VDD), L9.1 (VDD)
- net VDD: now also BACKLEDr1.2 (VDD), BACKLEDr10.2 (VDD), BACKLEDr11.2 (VDD), BACKLEDr12.2 (VDD), BACKLEDr13.2 (VDD), BACKLEDr14.2 (VDD), BACKLEDr15.2 (VDD), BACKLEDr16.2 (VDD), BACKLEDr17.2 (VDD), BACKLEDr18.2 (VDD), BACKLEDr2.2 (VDD), BACKLEDr3.2 (VDD), BACKLEDr4.2 (VDD), BACKLEDr5.2 (VDD), BACKLEDr6.2 (VDD), BACKLEDr7.2 (VDD), BACKLEDr8.2 (VDD), BACKLEDr9.2 (VDD), C2.1, L28.1 (VDD), L29.1 (VDD), L30.1 (VDD), L31.1 (VDD), L32.1 (VDD), L33.1 (VDD), L34.1 (VDD), L35.1 (VDD), L36.1 (VDD), L37.1 (VDD), L38.1 (VDD), L39.1 (VDD), L40.1 (VDD), L41.1 (VDD), L42.1 (VDD), L43.1 (VDD), L44.1 (VDD), L45.1 (VDD), L46.1 (VDD), L47.1 (VDD), L48.1 (VDD)
- net LED: now reaches U1.1 (TX0/D3)
- net LED: now also BACKLED1.1 (DIN)
- net LED_r: now reaches U2.1 (TX0/D3)
- net LED_r: now also BACKLEDr1.1 (DIN)
- new net: BACKLED17.3 (DOUT), BACKLED18.1 (DIN)
- new net: L11.3 (DIN), L5.2 (DOUT)
- new net: L5.3 (DIN), L6.2 (DOUT)
- new net: BACKLED15.3 (DOUT), BACKLED16.1 (DIN)
- new net: BACKLED16.3 (DOUT), BACKLED17.1 (DIN)
- new net: L43.3 (DIN), L46.2 (DOUT)
- new net: L46.3 (DIN), L47.2 (DOUT)
- new net: BACKLEDr15.3 (DOUT), BACKLEDr16.1 (DIN)
- new net: BACKLEDr16.3 (DOUT), BACKLEDr17.1 (DIN)
- new net: L31.3 (DIN), L37.2 (DOUT)
- new net: L37.3 (DIN), L43.2 (DOUT)
- new net: L1.3 (DIN), L2.2 (DOUT)
- new net: L2.3 (DIN), L8.2 (DOUT)
- new net: L1.2 (DOUT), L7.3 (DIN)
- new net: L29.3 (DIN), L35.2 (DOUT)
- new net: L35.3 (DIN), L41.2 (DOUT)
- new net: L30.2 (DOUT), L36.3 (DIN)
- new net: L30.3 (DIN), L31.2 (DOUT)
- new net: BACKLEDr13.3 (DOUT), BACKLEDr14.1 (DIN)
- new net: BACKLEDr14.3 (DOUT), BACKLEDr15.1 (DIN)
- new net: L10.3 (DIN), L16.2 (DOUT)
- new net: L16.3 (DIN), L19.2 (DOUT)
- new net: BACKLED12.3 (DOUT), BACKLED13.1 (DIN)
- new net: BACKLED13.3 (DOUT), BACKLED14.1 (DIN)
- new net: BACKLED14.3 (DOUT), BACKLED15.1 (DIN)
- new net: BACKLEDr5.3 (DOUT), BACKLEDr6.1 (DIN)
- new net: BACKLEDr6.3 (DOUT), BACKLEDr7.1 (DIN)
- new net: L28.2 (DOUT), L34.3 (DIN)
- new net: L28.3 (DIN), L29.2 (DOUT)
- new net: L14.3 (DIN), L15.2 (DOUT)
- new net: L15.3 (DIN), L9.2 (DOUT)
- new net: L34.2 (DOUT), L40.3 (DIN)
- new net: BACKLEDr4.3 (DOUT), BACKLEDr5.1 (DIN)
- new net: L11.2 (DOUT), L17.3 (DIN)
- new net: L38.2 (DOUT), L44.3 (DIN)
- new net: L32.2 (DOUT), L38.3 (DIN)
- new net: BACKLEDr17.3 (DOUT), BACKLEDr18.1 (DIN)
- new net: L10.2 (DOUT), L4.3 (DIN)
- new net: L14.2 (DOUT), L8.3 (DIN)
- new net: L3.2 (DOUT), L9.3 (DIN)
- new net: L3.3 (DIN), L4.2 (DOUT)
- new net: BACKLED3.3 (DOUT), BACKLED4.1 (DIN)
- new net: BACKLED4.3 (DOUT), BACKLED5.1 (DIN)
- new net: BACKLEDr7.3 (DOUT), BACKLEDr8.1 (DIN)
- new net: L39.3 (DIN), L45.2 (DOUT)
- new net: L45.3 (DIN), L48.2 (DOUT)
- new net: BACKLED10.3 (DOUT), BACKLED11.1 (DIN)
- new net: BACKLED11.3 (DOUT), BACKLED12.1 (DIN)
- new net: BACKLEDr8.3 (DOUT), BACKLEDr9.1 (DIN)
- new net: BACKLEDr10.1 (DIN), BACKLEDr9.3 (DOUT)
- new net: BACKLEDr1.3 (DOUT), BACKLEDr2.1 (DIN)
- new net: BACKLEDr2.3 (DOUT), BACKLEDr3.1 (DIN)
- new net: L19.3 (DIN), L20.2 (DOUT)
- new net: L17.2 (DOUT), L20.3 (DIN)
- new net: L41.3 (DIN), L42.2 (DOUT)
- new net: BACKLED6.3 (DOUT), BACKLED7.1 (DIN)
- new net: BACKLED7.3 (DOUT), BACKLED8.1 (DIN)
- new net: BACKLEDr3.3 (DOUT), BACKLEDr4.1 (DIN)
- new net: BACKLED8.3 (DOUT), BACKLED9.1 (DIN)
- new net: L13.3 (DIN), L7.2 (DOUT)
- new net: BACKLED10.1 (DIN), BACKLED9.3 (DOUT)
- new net: L44.2 (DOUT), L47.3 (DIN)
- new net: BACKLEDr11.3 (DOUT), BACKLEDr12.1 (DIN)
- new net: BACKLEDr12.3 (DOUT), BACKLEDr13.1 (DIN)
- new net: BACKLED5.3 (DOUT), BACKLED6.1 (DIN)
- new net: L18.3 (DIN), L21.2 (DOUT)
- new net: BACKLEDr10.3 (DOUT), BACKLEDr11.1 (DIN)
- new net: BACKLED1.3 (DOUT), BACKLED2.1 (DIN)
- new net: L32.3 (DIN), L33.2 (DOUT)
- new net: L33.3 (DIN), L39.2 (DOUT)
- new net: L12.2 (DOUT), L6.3 (DIN)
- new net: L12.3 (DIN), L18.2 (DOUT)
- new net: BACKLED2.3 (DOUT), BACKLED3.1 (DIN)
- new net: L36.2 (DOUT), L42.3 (DIN)
- new net LED_CONT: BACKLED18.3 (DOUT), L21.3 (DIN)
- new net LEDr_CONT: BACKLEDr18.3 (DOUT), L48.3 (DIN)
Other:
- moved on the sheet: D1, D10, D11, D12, D13, D14, D15, D16, D17, D18, D19, D2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
