File: sweeq mx/sweeq mx.kicad_pcb (KiCad board)
At the start: 2 copper layers, 231.1 x 95.2 mm, 88 parts, among them J1 MJ-4PP-9, J2 MJ-4PP-9, SW1 SW_PUSH, SW10 SW_PUSH, SW11 SW_PUSH, SW12 SW_PUSH, SW13 SW_PUSH, SW14 SW_PUSH, SW15 SW_PUSH, SW16 SW_PUSH, SW17 SW_PUSH, SW18 SW_PUSH, SW19 SW_PUSH, SW2 SW_PUSH, SW20 SW_PUSH, SW21 SW_PUSH, SW22 SW_PUSH, SW23 SW_PUSH, SW24 SW_PUSH, SW25 SW_PUSH, SW26 SW_PUSH, SW27 SW_PUSH, SW28 SW_PUSH, SW29 SW_PUSH, SW3 SW_PUSH, SW30 SW_PUSH, SW31 SW_PUSH, SW32 SW_PUSH, SW33 SW_PUSH, SW34 SW_PUSH, SW4 SW_PUSH, SW5 SW_PUSH, SW6 SW_PUSH, SW7 SW_PUSH, SW8 SW_PUSH, SW9 SW_PUSH, U1 ProMicro, U2 ProMicro

Commit message: sweeq mx: bump version
Other:
- board text added: "755a6e6"
- board text removed: "0fc7c04"

Commit message: sweeq mx: add tabs
Parts:
- added REF**: Tab, kikit:Tab, B.Cu at (-79.4, 32.8)
- added REF**: Tab, kikit:Tab, B.Cu at (-30.8, -62.8)
- added REF**: Tab, kikit:Tab, F.Cu at (-170.1, 50.7)
- added REF**: Tab, kikit:Tab, F.Cu at (-125.9, -63.3)
- added REF**: Tab, kikit:Tab, F.Cu at (-169.3, -44.8)
- added REF**: Tab, kikit:Tab, F.Cu at (-120.6, 50.7)
- added REF**: Tab, kikit:Tab, B.Cu at (-36.1, 51.2)
- added REF**: Tab, kikit:Tab, B.Cu at (-80.2, -62.8)
- moved D1 342.8 mm to (-68.3, -60.3), turned to 180 degrees
- moved SW1 337.0 mm to (-74.0, -53.0), turned to -90 degrees
- moved Mounting 04 335.2 mm to (-84.7, -45.8), turned to 90 degrees
- moved D6 332.7 mm to (-49.1, -60.5), turned to 180 degrees
- moved D2 326.7 mm to (-79.6, -41.8), turned to 180 degrees
- moved SW6 325.9 mm to (-55.0, -53.0), turned to -90 degrees
- moved D11 325.8 mm to (-34.8, -60.2), turned to 180 degrees
- moved SW2 321.8 mm to (-86.0, -34.0), turned to -90 degrees
- moved SW11 316.6 mm to (-36.0, -53.0), turned to -90 degrees
- moved D7 314.4 mm to (-61.0, -41.5), turned to 180 degrees
- moved SW7 308.6 mm to (-66.9, -34.0), turned to -90 degrees
- moved D3 308.3 mm to (-86.1, -22.7), turned to 180 degrees
- moved D12 304.5 mm to (-43.2, -41.4), turned to 180 degrees
- moved SW3 304.2 mm to (-92.1, -15.0), turned to -90 degrees
- moved J2 302.6 mm to (-122.2, -61.9), turned to 0 degrees
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Other:
- board size 231.1 x 95.2 mm -> 185 x 113.9 mm
