File: corne/corne-cherry/pcb/corne-cherry.kicad_pcb (KiCad board)
At the start: 2 copper layers, 274.5 x 91.4 mm, 110 parts, among them J1 MJ-4PP-9, J2 OLED, J3 MJ-4PP-9, J4 OLED, SW1 SW_PUSH, SW10 SW_PUSH, SW11 SW_PUSH, SW12 SW_PUSH, SW13 SW_PUSH, SW14 SW_PUSH, SW15 SW_PUSH, SW16 SW_PUSH, SW17 SW_PUSH, SW18 SW_PUSH, SW19 SW_PUSH, SW2 SW_PUSH, SW20 SW_PUSH, SW21 SW_PUSH, SW22 SW_PUSH, SW23 SW_PUSH, SW24 SW_PUSH, SW25 SW_PUSH, SW26 SW_PUSH, SW27 SW_PUSH, SW28 SW_PUSH, SW29 SW_PUSH, SW3 SW_PUSH, SW30 SW_PUSH, SW31 SW_PUSH, SW32 SW_PUSH, SW33 SW_PUSH, SW34 SW_PUSH, SW35 SW_PUSH, SW36 SW_PUSH, SW37 SW_PUSH, SW38 SW_PUSH, SW39 SW_PUSH, SW4 SW_PUSH, SW40 SW_PUSH, SW41 SW_PUSH, SW42 SW_PUSH, SW5 SW_PUSH, SW6 SW_PUSH, SW7 SW_PUSH, SW8 SW_PUSH, SW9 SW_PUSH, U1 ProMicro, U2 ProMicro

Commit message: corne/cherry: fix m2 holes, we need the spacer to go through them
Parts:
- added REF**: logo big, holykeebs:logo .5x, B.Cu at (134.4, 41.5)
- added REF**: logo big, holykeebs:logo .5x, B.Cu at (162.0, 41.5)
- Ref** (x10): footprint holykeebs:M2_HOLE_NPH -> holykeebs:M2_HOLE_NPH_BIG
Connections:
- D1 pad 2: (no net) -> Net-(D1-A)
- D10 pad 2: (no net) -> Net-(D10-A)
- D11 pad 2: (no net) -> Net-(D11-A)
- D12 pad 2: (no net) -> Net-(D12-A)
- D13 pad 2: (no net) -> Net-(D13-A)
- D14 pad 2: (no net) -> Net-(D14-A)
- D15 pad 2: (no net) -> Net-(D15-A)
- D16 pad 2: (no net) -> Net-(D16-A)
- D17 pad 2: (no net) -> Net-(D17-A)
- D18 pad 2: (no net) -> Net-(D18-A)
- D19 pad 2: (no net) -> Net-(D19-A)
- D2 pad 2: (no net) -> Net-(D2-A)
- D20 pad 2: (no net) -> Net-(D20-A)
- D21 pad 2: (no net) -> Net-(D21-A)
- D22 pad 2: (no net) -> Net-(D22-A)
- D23 pad 2: (no net) -> Net-(D23-A)
- D24 pad 2: (no net) -> Net-(D24-A)
- D25 pad 2: (no net) -> Net-(D25-A)
- D26 pad 2: (no net) -> Net-(D26-A)
- D27 pad 2: (no net) -> Net-(D27-A)
- D28 pad 2: (no net) -> Net-(D28-A)
- D29 pad 2: (no net) -> Net-(D29-A)
- D3 pad 2: (no net) -> Net-(D3-A)
- D30 pad 2: (no net) -> Net-(D30-A)
- D31 pad 2: (no net) -> Net-(D31-A)
- D32 pad 2: (no net) -> Net-(D32-A)
- D33 pad 2: (no net) -> Net-(D33-A)
- D34 pad 2: (no net) -> Net-(D34-A)
- D35 pad 2: (no net) -> Net-(D35-A)
- D36 pad 2: (no net) -> Net-(D36-A)
- D37 pad 2: (no net) -> Net-(D37-A)
- D38 pad 2: (no net) -> Net-(D38-A)
- D39 pad 2: (no net) -> Net-(D39-A)
- D4 pad 2: (no net) -> Net-(D4-A)
- D40 pad 2: (no net) -> Net-(D40-A)
- D41 pad 2: (no net) -> Net-(D41-A)
- D42 pad 2: (no net) -> Net-(D42-A)
- D5 pad 2: (no net) -> Net-(D5-A)
- D6 pad 2: (no net) -> Net-(D6-A)
- D7 pad 2: (no net) -> Net-(D7-A)
- D8 pad 2: (no net) -> Net-(D8-A)
- D9 pad 2: (no net) -> Net-(D9-A)
- J1 pad A: (no net) -> unconnected-(J1-PadA)
- J3 pad A: (no net) -> unconnected-(J3-PadA)
- U1 pad 11: (no net) -> unconnected-(U1-8/B4-Pad11)
- U1 pad 12: (no net) -> unconnected-(U1-9/B5-Pad12)
- U1 pad 13: (no net) -> unconnected-(U1-B6/10-Pad13)
- U1 pad 14: (no net) -> unconnected-(U1-B2/16-Pad14)
- U1 pad 24: (no net) -> unconnected-(U1-RAW-Pad24)
- U2 pad 11: (no net) -> unconnected-(U2-8/B4-Pad11)
- U2 pad 12: (no net) -> unconnected-(U2-9/B5-Pad12)
- U2 pad 13: (no net) -> unconnected-(U2-B6/10-Pad13)
- U2 pad 14: (no net) -> unconnected-(U2-B2/16-Pad14)
- U2 pad 24: (no net) -> unconnected-(U2-RAW-Pad24)
Routing:
- net GNDA: track 61.6 -> 70.6 mm
- net data_r: track 62.9 -> 61.9 mm
- net VCC: track 48.8 -> 48.1 mm
- net Net-(D39-A): track 4.68 -> 4.04 mm

Commit message: corne/cherry: bump version
Other:
- board text added: "65be52c"

Commit message: corne cherry: changes?
Parts:
- U1, U2: footprint kbd:ProMicro_v3 -> holykeebs:ProMicro_1mm_holes
