File: lily58/choc smt/Lily58.kicad_pcb (KiCad board)
At the start: 2 copper layers, 279.3 x 99.1 mm, 152 parts, among them J1 4PIN, J2 4PIN, P1 OLED, P2 OLED, SW1 SW_PUSH, SW10 SW_PUSH, SW11 SW_PUSH, SW12 SW_PUSH, SW13 SW_PUSH, SW14 SW_PUSH, SW15 SW_PUSH, SW16 SW_PUSH, SW17 SW_PUSH, SW18 SW_PUSH, SW19 SW_PUSH, SW2 SW_PUSH, SW20 SW_PUSH, SW21 SW_PUSH, SW22 SW_PUSH, SW23 SW_PUSH, SW24 SW_PUSH, SW25 SW_PUSH, SW26 SW_PUSH, SW27 SW_PUSH, SW28 SW_PUSH, SW29 SW_PUSH, SW3 SW_PUSH, SW30 SW_PUSH, SW31 SW_PUSH, SW32 SW_PUSH, SW33 SW_PUSH, SW34 SW_PUSH, SW35 SW_PUSH, SW36 SW_PUSH, SW37 SW_PUSH, SW38 SW_PUSH, SW39 SW_PUSH, SW4 SW_PUSH, SW40 SW_PUSH, SW41 SW_PUSH, SW42 SW_PUSH, SW43 SW_PUSH, SW44 SW_PUSH, SW45 SW_PUSH, SW46 SW_PUSH, SW47 SW_PUSH, SW48 SW_PUSH, SW49 SW_PUSH, SW5 SW_PUSH, SW50 SW_PUSH, SW51 SW_PUSH, SW52 SW_PUSH, SW53 SW_PUSH, SW54 SW_PUSH, SW55 SW_PUSH, SW56 SW_PUSH, SW57 SW_PUSH, SW58 SW_PUSH, SW6 SW_PUSH, SW7 SW_PUSH, SW8 SW_PUSH, SW9 SW_PUSH, U1 ProMicro, U2 ProMicro

Commit message: lily58 choc: bump version
Other:
- board text added: "056af16"
- board text removed: "8c8d947"

Commit message: lily58 choc: move top edge and 1.5u key
Parts:
- removed the REF** at (347.4, 143.8)
- removed the REF** at (225.3, 219.8)
- removed the REF** at (225.8, 146.0)
- added REF**: Tab, kikit:Tab, B.Cu at (235.8, 219.9)
- added REF**: Tab, kikit:Tab, B.Cu at (225.9, 144.9)
- added REF**: Tab, kikit:Tab, B.Cu at (346.6, 142.8)
- moved REF** 10.4 mm to (192.2, 219.9)
- moved REF** 1.26 mm to (81.4, 142.8)
- moved REF** 1.03 mm to (202.1, 144.9)
- moved SW55 0.50 mm to (331.7, 226.8)
- moved SW26 0.50 mm to (96.3, 226.8)
Other:
- board size 279.3 x 99.1 mm -> 279.3 x 100.1 mm

Commit message: lily58 choc: move trrs jack to the edge
Parts:
- moved J1 2.20 mm to (79.4, 143.2)
- moved J2 2.20 mm to (348.6, 143.2)
