File: lily58/choc smt/Lily58.kicad_pcb (KiCad board)
At the start: 2 copper layers, 279.3 x 100.1 mm, 152 parts, among them J1 4PIN, J2 4PIN, P1 OLED, P2 OLED, SW1 SW_PUSH, SW10 SW_PUSH, SW11 SW_PUSH, SW12 SW_PUSH, SW13 SW_PUSH, SW14 SW_PUSH, SW15 SW_PUSH, SW16 SW_PUSH, SW17 SW_PUSH, SW18 SW_PUSH, SW19 SW_PUSH, SW2 SW_PUSH, SW20 SW_PUSH, SW21 SW_PUSH, SW22 SW_PUSH, SW23 SW_PUSH, SW24 SW_PUSH, SW25 SW_PUSH, SW26 SW_PUSH, SW27 SW_PUSH, SW28 SW_PUSH, SW29 SW_PUSH, SW3 SW_PUSH, SW30 SW_PUSH, SW31 SW_PUSH, SW32 SW_PUSH, SW33 SW_PUSH, SW34 SW_PUSH, SW35 SW_PUSH, SW36 SW_PUSH, SW37 SW_PUSH, SW38 SW_PUSH, SW39 SW_PUSH, SW4 SW_PUSH, SW40 SW_PUSH, SW41 SW_PUSH, SW42 SW_PUSH, SW43 SW_PUSH, SW44 SW_PUSH, SW45 SW_PUSH, SW46 SW_PUSH, SW47 SW_PUSH, SW48 SW_PUSH, SW49 SW_PUSH, SW5 SW_PUSH, SW50 SW_PUSH, SW51 SW_PUSH, SW52 SW_PUSH, SW53 SW_PUSH, SW54 SW_PUSH, SW55 SW_PUSH, SW56 SW_PUSH, SW57 SW_PUSH, SW58 SW_PUSH, SW6 SW_PUSH, SW7 SW_PUSH, SW8 SW_PUSH, SW9 SW_PUSH, U1 ProMicro, U2 ProMicro

Commit message: lily choc: move mounting holes
Parts:
- moved TH4 17.9 mm to (192.9, 156.6)
- moved TH4 17.9 mm to (235.1, 156.6)
- moved TH3 16.6 mm to (120.8, 152.4)
- moved TH3 16.6 mm to (307.2, 152.4)
- moved D2 2.88 mm to (124.3, 148.8)
- moved D6 2.61 mm to (196.3, 154.2)
- moved D31 2.32 mm to (303.9, 149.0)
- moved D35 1.72 mm to (231.2, 153.8)
Routing:
- net GND: track 72.8 -> 76.5 mm
- net row0: track 111.7 -> 115.2 mm
- net col1_l: track 217.6 -> 221.1 mm
- net DATA_l: track 7.66 -> 11.0 mm
- net Net-(D2-A): track 5.76 -> 8.38 mm
- net RESET: track 29.5 -> 32.1 mm
- net row0_l: track 128.0 -> 130.5 mm
- net GNDA: track 76.4 -> 74.1 mm
- net Net-(D6-A): track 7.24 -> 8.77 mm
- net DATA: track 19.5 -> 20.5 mm
- net VCC: track 32.3 -> 33.2 mm
- net VDD: track 66.8 -> 67.7 mm
- net col3_l: track 182.5 -> 183.3 mm
- net col4_l: track 178.4 -> 179.2 mm
- net col0_l: track 190.0 -> 190.8 mm
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
Commit message: lily choc: bump version
Other:
- board text added: "d1c2c10"
- board text removed: "056af16"
